File: PIC18F24K40.sch (KiCad schematic (older format))
At the start: 15 parts, among them J1 Conn_01x13, J2 Conn_01x13, J3 ICSP, J4 USB_B_Micro, U1 FT231XQ, U2 PIC18F24K40-I_ML

Commit message: Reset button added Designators hidden
Parts:
- added SW1: SW_SPST, _PIC18F24K40:SW_SPST_B3U-1000P, symbol _PIC18F24K40:SW_SPST
Connections:
- wire segments 105 -> 107
Changed lines of the file:
@@
 	6000 1650 6650 1650
 Connection ~ 6650 2400
+Text Notes 7900 4550 0    50   ~ 0
+Alternate part number for female header:\nPPTC131LFBN-RC
+Text Notes 8100 3150 0    50   ~ 0
+Alternate part number for right angle\nPRPC006SBAN-M71RC
+$Comp
+L _PIC18F24K40:SW_SPST SW1
+U 1 1 5BD32462
+P 3700 5900
+F 0 "SW1" V 3750 6200 50  0000 R CNN
+F 1 "SW_SPST" V 3600 6300 50  0000 R CNN
+F 2 "_PIC18F24K40:SW_SPST_B3U-1000P" H 3700 5900 50  0001 C CNN
+F 3 "" H 3700 5900 50  0001 C CNN
+	1    3700 5900
+	0    -1   -1   0
+$EndComp
+$Comp
+L _PIC18F24K40:GND #PWR01
+U 1 1 5BD325E7
+P 3700 6150
+F 0 "#PWR01" H 3700 5900 50  0001 C CNN
+F 1 "GND" H 3705 5977 50  0000 C CNN
+F 2 "" H 3700 6150 50  0001 C CNN
+F 3 "" H 3700 6150 50  0001 C CNN
+	1    3700 6150
+	1    0    0    -1
+$EndComp
+Wire Wire Line
+	3700 6150 3700 6100
+Wire Wire Line
+	3700 5700 3700 5650
 Wire Bus Line
 	6400 5750 6400 6550
@@
 Wire Bus Line
 	3400 4100 3400 5650
-Text Notes 7900 4550 0    50   ~ 0
-Alternate part number for female header:\nPPTC131LFBN-RC
-Text Notes 8100 3150 0    50   ~ 0
-Alternate part number for right angle\nPRPC006SBAN-M71RC
+Connection ~ 3700 5650
 $EndSCHEMATC

Commit message: Ordering details added for push button
Parts:
- SW1: Manufacturer (none) -> Omron Electronics Inc-EMC Div; Manufacturer Part Number (none) -> B3U-1000P
Changed lines of the file:
@@
 F 2 "_PIC18F24K40:SW_SPST_B3U-1000P" H 3700 5900 50  0001 C CNN
 F 3 "" H 3700 5900 50  0001 C CNN
+F 4 "Omron Electronics Inc-EMC Div" H 0   0   50  0001 C CNN "Manufacturer"
+F 5 "B3U-1000P" H 0   0   50  0001 C CNN "Manufacturer Part Number"
 	1    3700 5900
 	0    -1   -1   0
@@
 Wire Wire Line
 	3700 5700 3700 5650
+Connection ~ 3700 5650
 Wire Bus Line
 	6400 5750 6400 6550
@@
 Wire Bus Line
 	3400 4100 3400 5650
-Connection ~ 3700 5650
 $EndSCHEMATC

Commit message: LED and phototransistor added
I've added an LED for output and phototransistor for input. No button
though.
Parts:
- added C6: 0.01uf, _PIC18F24K40:C_0603_1608Metric_Pad1.05x0.95mm_HandSolder, symbol _PIC18F24K40:C_Small
- added D1: blue, _PIC18F24K40:LED_0603_1608Metric, symbol _PIC18F24K40:LED_Small
- added Q1: Q_Photo_NPN, _PIC18F24K40:LED_0603_1608Metric, symbol _PIC18F24K40:Q_Photo_NPN
- added R4: 360, _PIC18F24K40:R_0603_1608Metric_Pad1.05x0.95mm_HandSolder, symbol _PIC18F24K40:R_Small_US
- added R5: 10k, _PIC18F24K40:R_0603_1608Metric_Pad1.05x0.95mm_HandSolder, symbol _PIC18F24K40:R_Small_US
Connections:
- wire segments 107 -> 118
Changed lines of the file:
@@
 $EndComp
 Wire Bus Line
-	6400 4100 7050 4100
+	6400 3750 7500 3750
 Entry Wire Line
 	6300 4550 6400 4650
@@
 	3300 5450 2950 5450
 Wire Wire Line
-	3300 5550 2950 5550
-Entry Wire Line
-	7050 4550 7150 4650
-Entry Wire Line
-	7050 4650 7150 4750
-Entry Wire Line
-	7050 4750 7150 4850
-Entry Wire Line
-	7050 4850 7150 4950
-Entry Wire Line
-	7050 4950 7150 5050
-Entry Wire Line
-	7050 5050 7150 5150
-Entry Wire Line
-	7050 5150 7150 5250
-Entry Wire Line
-	7050 5250 7150 5350
-Entry Wire Line
-	7050 5350 7150 5450
-Entry Wire Line
-	7050 5450 7150 5550
-Entry Wire Line
-	7050 5550 7150 5650
-Wire Wire Line
-	7600 4650 7150 4650
-Wire Wire Line
-	7150 4750 7600 4750
-Wire Wire Line
-	7600 4850 7150 4850
-Wire Wire Line
-	7150 4950 7600 4950
-Wire Wire Line
-	7600 5050 7150 5050
-Wire Wire Line
-	7150 5150 7600 5150
-Wire Wire Line
-	7600 5250 7150 5250
-Wire Wire Line
-	7150 5350 7600 5350
-Wire Wire Line
-	7600 5450 7150 5450
-Wire Wire Line
-	7150 5550 7600 5550
-Wire Wire Line
-	7600 5650 7150 5650
+	3300 5550 3000 5550
+Entry Wire Line
+	7500 4200 7600 4300
+Entry Wire Line
+	7500 4300 7600 4400
+Entry Wire Line
+	7500 4400 7600 4500
+Entry Wire Line
+	7500 4500 7600 4600
+Entry Wire Line
+	7500 4600 7600 4700
+Entry Wire Line
+	7500 4700 7600 4800
+Entry Wire Line
+	7500 4800 7600 4900
+Entry Wire Line
+	7500 4900 7600 5000
+Entry Wire Line
+	7500 5000 7600 5100
+Entry Wire Line
+	7500 5100 7600 5200
+Entry Wire Line
+	7500 5200 7600 5300
+Wire Wire Line
+	8050 4300 7600 4300
+Wire Wire Line
+	7600 4400 8050 4400
+Wire Wire Line
+	8050 4500 7600 4500
+Wire Wire Line
+	7600 4600 8050 4600
+Wire Wire Line
+	8050 4700 7600 4700
+Wire Wire Line
+	7600 4800 8050 4800
+Wire Wire Line
+	8050 4900 7600 4900
+Wire Wire Line
+	7600 5000 8050 5000
+Wire Wire Line
+	8050 5100 7600 5100
+Wire Wire Line
+	7600 5200 8050 5200
 Text Label 4300 4700 0    50   ~ 0
 RA0
@@
 Text Label 3050 5550 0    50   ~ 0
 RC4
-Text Label 7350 5650 0    50   ~ 0
+Text Label 7800 5300 0    50   ~ 0
 RC5
-Text Label 7350 5550 0    50   ~ 0
+Text Label 7800 5200 0    50   ~ 0
 RC6
-Text Label 7350 5450 0    50   ~ 0
+Text Label 7800 5100 0    50   ~ 0
 RC7
-Text Label 7350 5350 0    50   ~ 0
+Text Label 7800 5000 0    50   ~ 0
 RB0
-Text Label 7350 5250 0    50   ~ 0
+Text Label 7800 4900 0    50   ~ 0
 RB1
-Text Label 7350 5150 0    50   ~ 0
+Text Label 7800 4800 0    50   ~ 0
 RB2
-Text Label 7350 5050 0    50   ~ 0
+Text Label 7800 4700 0    50   ~ 0
 RB3
-Text Label 7350 4950 0    50   ~ 0
+Text Label 7800 4600 0    50   ~ 0
 RB4
-Text Label 7350 4850 0    50   ~ 0
+Text Label 7800 4500 0    50   ~ 0
 RB5
-Text Label 7350 4750 0    50   ~ 0
+Text Label 7800 4400 0    50   ~ 0
 RB6
-Text Label 7350 4650 0    50   ~ 0
+Text Label 7800 4300 0    50   ~ 0
 RB7
 $Comp
@@
 L _PIC18F24K40:Conn_01x13 J2
 U 1 1 5BD14518
-P 7800 5050
-F 0 "J2" H 7880 5092 50  0000 L CNN
-F 1 "Conn_01x13" H 7880 5001 50  0000 L CNN
-F 2 "_PIC18F24K40:PinHeader_1x13_P2.54mm_Vertical" H 7800 5050 50  0001 C CNN
-F 3 "~" H 7800 5050 50  0001 C CNN
-F 4 "Sullins Connector Solutions" H 800 650 50  0001 C CNN "Manufacturer"
-F 5 "PREC013SAAN-RC" H 800 650 50  0001 C CNN "Manufacturer Part Number"
-	1    7800 5050
+P 8250 4700
+F 0 "J2" H 8330 4742 50  0000 L CNN
+F 1 "Conn_01x13" H 8330 4651 50  0000 L CNN
+F 2 "_PIC18F24K40:PinHeader_1x13_P2.54mm_Vertical" H 8250 4700 50  0001 C CNN
+F 3 "~" H 8250 4700 50  0001 C CNN
+F 4 "Sullins Connector Solutions" H 1250 300 50  0001 C CNN "Manufacturer"
+F 5 "PREC013SAAN-RC" H 1250 300 50  0001 C CNN "Manufacturer Part Number"
+	1    8250 4700
 	1    0    0    -1
 $EndComp
@@
 L _PIC18F24K40:GND #PWR0102
 U 1 1 5BD1690C
-P 7400 4550
-F 0 "#PWR0102" H 7400 4300 50  0001 C CNN
-F 1 "GND" V 7405 4377 50  0000 C CNN
-F 2 "" H 7400 4550 50  0001 C CNN
-F 3 "" H 7400 4550 50  0001 C CNN
-	1    7400 4550
+P 7850 4200
+F 0 "#PWR0102" H 7850 3950 50  0001 C CNN
+F 1 "GND" V 7855 4027 50  0000 C CNN
+F 2 "" H 7850 4200 50  0001 C CNN
+F 3 "" H 7850 4200 50  0001 C CNN
+	1    7850 4200
 	0    1    1    0
 $EndComp
 Wire Wire Line
-	7600 4550 7400 4550
+	8050 4200 7850 4200
 $Comp
 L _PIC18F24K40:GND #PWR0104
@@
 L _PIC18F24K40:+5v_USB #PWR0106
 U 1 1 5BDB1C98
-P 7550 4450
-F 0 "#PWR0106" H 7550 4300 50  0001 C CNN
-F 1 "+5v_USB" V 7568 4578 50  0000 L CNN
-F 2 "" H 7550 4450 50  0001 C CNN
-F 3 "" H 7550 4450 50  0001 C CNN
-	1    7550 4450
+P 8000 4100
+F 0 "#PWR0106" H 8000 3950 50  0001 C CNN
+F 1 "+5v_USB" V 8018 4228 50  0000 L CNN
+F 2 "" H 8000 4100 50  0001 C CNN
+F 3 "" H 8000 4100 50  0001 C CNN
+	1    8000 4100
 	0    -1   -1   0
 $EndComp
 Wire Wire Line
-	7600 4450 7550 4450
+	8050 4100 8000 4100
 $Comp
 L _PIC18F24K40:+5v_USB #PWR0107
@@
 	6000 1650 6650 1650
 Connection ~ 6650 2400
-Text Notes 7900 4550 0    50   ~ 0
+Text Notes 8400 4450 0    50   ~ 0
 Alternate part number for female header:\nPPTC131LFBN-RC
 Text Notes 8100 3150 0    50   ~ 0
@@
 	3700 5700 3700 5650
 Connection ~ 3700 5650
+$Comp
+L _PIC18F24K40:LED_Small D1
+U 1 1 5BD5F206
+P 3000 6000
+F 0 "D1" V 3046 5932 50  0000 R CNN
+F 1 "blue" V 2950 6500 50  0000 R CNN
+F 2 "_PIC18F24K40:LED_0603_1608Metric" V 3000 6000 50  0001 C CNN
+F 3 "~" V 3000 6000 50  0001 C CNN
+F 4 "Everlight Electronics Co Ltd" H 0   0   50  0001 C CNN "Manufacturer"
+F 5 "19-213SUBC/S400-A5/S208-2/TR8" H 0   0   50  0001 C CNN "Manufacturer Part Number"
+	1    3000 6000
+	0    -1   -1   0
+$EndComp
+Wire Wire Line
+	3000 5900 3000 5550
+Connection ~ 3000 5550
+Wire Wire Line
+	3000 5550 2950 5550
+$Comp
+L _PIC18F24K40:GND #PWR03
+U 1 1 5BD63C57
+P 3000 6400
+F 0 "#PWR03" H 3000 6150 50  0001 C CNN
+F 1 "GND" H 3005 6227 50  0000 C CNN
+F 2 "" H 3000 6400 50  0001 C CNN
+F 3 "" H 3000 6400 50  0001 C CNN
+	1    3000 6400
+	1    0    0    -1
+$EndComp
+$Comp
+L _PIC18F24K40:R_Small_US R4
+U 1 1 5BD63EAC
+P 3000 6250
+F 0 "R4" H 3068 6296 50  0000 L CNN
+F 1 "360" H 3068 6205 50  0000 L CNN
+F 2 "_PIC18F24K40:R_0603_1608Metric_Pad1.05x0.95mm_HandSolder" H 3000 6250 50  0001 C CNN
+F 3 "~" H 3000 6250 50  0001 C CNN
+	1    3000 6250
+	1    0    0    -1
+$EndComp
+Wire Wire Line
+	3000 6100 3000 6150
+Wire Wire Line
+	3000 6350 3000 6400
+$Comp
+L _PIC18F24K40:Q_Photo_NPN Q1
+U 1 1 5BD727A9
+P 7150 5850
+F 0 "Q1" H 7340 5896 50  0000 L CNN
+F 1 "Q_Photo_NPN" H 7340 5805 50  0000 L CNN
+F 2 "_PIC18F24K40:LED_0603_1608Metric" H 7350 5950 50  0001 C CNN
+F 3 "~" H 7150 5850 50  0001 C CNN
+F 4 "Everlight Electronics Co Ltd" H 450 -350 50  0001 C CNN "Manufacturer"
+F 5 "PT19-21B/L41/TR8" H 450 -350 50  0001 C CNN "Manufacturer Part Number"
+	1    7150 5850
+	1    0    0    -1
+$EndComp
+$Comp
+L _PIC18F24K40:GND #PWR04
+U 1 1 5BD7297F
+P 7250 6150
+F 0 "#PWR04" H 7250 5900 50  0001 C CNN
+F 1 "GND" H 7255 5977 50  0000 C CNN
+F 2 "" H 7250 6150 50  0001 C CNN
+F 3 "" H 7250 6150 50  0001 C CNN
+	1    7250 6150
+	1    0    0    -1
+$EndComp
+Wire Wire Line
+	7250 6150 7250 6050
+$Comp
+L _PIC18F24K40:R_Small_US R5
+U 1 1 5BD775F5
+P 8000 5450
+F 0 "R5" H 7932 5404 50  0000 R CNN
+F 1 "10k" H 7932 5495 50  0000 R CNN
+F 2 "_PIC18F24K40:R_0603_1608Metric_Pad1.05x0.95mm_HandSolder" H 8000 5450 50  0001 C CNN
+F 3 "~" H 8000 5450 50  0001 C CNN
+	1    8000 5450
+	-1   0    0    1
+$EndComp
+Wire Wire Line
+	7250 5550 7250 5650
+$Comp
+L _PIC18F24K40:C_Small C6
+U 1 1 5BD82600
+P 8000 5850
+F 0 "C6" H 8092 5896 50  0000 L CNN
+F 1 "0.01uf" H 8092 5805 50  0000 L CNN
+F 2 "_PIC18F24K40:C_0603_1608Metric_Pad1.05x0.95mm_HandSolder" H 8000 5850 50  0001 C CNN
+F 3 "~" H 8000 5850 50  0001 C CNN
+	1    8000 5850
+	1    0    0    -1
+$EndComp
+$Comp
+L _PIC18F24K40:GND #PWR05
+U 1 1 5BD82668
+P 8000 6000
+F 0 "#PWR05" H 8000 5750 50  0001 C CNN
+F 1 "GND" H 8005 5827 50  0000 C CNN
+F 2 "" H 8000 6000 50  0001 C CNN
+F 3 "" H 8000 6000 50  0001 C CNN
+	1    8000 6000
+	1    0    0    -1
+$EndComp
+Wire Wire Line
+	8000 6000 8000 5950
+Wire Wire Line
+	7600 5300 8000 5300
+Wire Wire Line
+	7250 5550 8000 5550
+Wire Wire Line
+	8000 5550 8000 5750
+Connection ~ 8000 5550
+Wire Wire Line
+	8000 5350 8000 5300
+Connection ~ 8000 5300
+Wire Wire Line
+	8000 5300 8050 5300
 Wire Bus Line
 	6400 5750 6400 6550
@@
 	4000 4100 4000 6550
 Wire Bus Line
-	6400 4100 6400 5650
+	6400 3750 6400 5650
 Wire Bus Line
-	7050 4100 7050 5550
+	7500 3750 7500 5200
 Wire Bus Line
 	3400 4100 3400 5650

Commit message: RC5 now connected to the right place
OMG I screwed up the light sensor connection! The boards come in soon...

Schematic and board updated. Will kynar the prototypes
Connections:
- wire segments 118 -> 120
Other:
- moved on the sheet: C6
Changed lines of the file:
@@
 L _PIC18F24K40:Q_Photo_NPN Q1
 U 1 1 5BD727A9
-P 7150 5850
-F 0 "Q1" H 7340 5896 50  0000 L CNN
-F 1 "Q_Photo_NPN" H 7340 5805 50  0000 L CNN
-F 2 "_PIC18F24K40:LED_0603_1608Metric" H 7350 5950 50  0001 C CNN
-F 3 "~" H 7150 5850 50  0001 C CNN
-F 4 "Everlight Electronics Co Ltd" H 450 -350 50  0001 C CNN "Manufacturer"
-F 5 "PT19-21B/L41/TR8" H 450 -350 50  0001 C CNN "Manufacturer Part Number"
-	1    7150 5850
+P 6600 5950
+F 0 "Q1" H 6790 5996 50  0000 L CNN
+F 1 "Q_Photo_NPN" H 6800 5850 50  0001 L CNN
+F 2 "_PIC18F24K40:LED_0603_1608Metric" H 6800 6050 50  0001 C CNN
+F 3 "~" H 6600 5950 50  0001 C CNN
+F 4 "Everlight Electronics Co Ltd" H -100 -250 50  0001 C CNN "Manufacturer"
+F 5 "PT19-21B/L41/TR8" H -100 -250 50  0001 C CNN "Manufacturer Part Number"
+	1    6600 5950
 	1    0    0    -1
 $EndComp
@@
 L _PIC18F24K40:GND #PWR04
 U 1 1 5BD7297F
-P 7250 6150
-F 0 "#PWR04" H 7250 5900 50  0001 C CNN
-F 1 "GND" H 7255 5977 50  0000 C CNN
-F 2 "" H 7250 6150 50  0001 C CNN
-F 3 "" H 7250 6150 50  0001 C CNN
-	1    7250 6150
+P 6700 6250
+F 0 "#PWR04" H 6700 6000 50  0001 C CNN
+F 1 "GND" H 6705 6077 50  0000 C CNN
+F 2 "" H 6700 6250 50  0001 C CNN
+F 3 "" H 6700 6250 50  0001 C CNN
+	1    6700 6250
 	1    0    0    -1
 $EndComp
 Wire Wire Line
-	7250 6150 7250 6050
+	6700 6250 6700 6150
 $Comp
 L _PIC18F24K40:R_Small_US R5
 U 1 1 5BD775F5
-P 8000 5450
-F 0 "R5" H 7932 5404 50  0000 R CNN
-F 1 "10k" H 7932 5495 50  0000 R CNN
-F 2 "_PIC18F24K40:R_0603_1608Metric_Pad1.05x0.95mm_HandSolder" H 8000 5450 50  0001 C CNN
-F 3 "~" H 8000 5450 50  0001 C CNN
-	1    8000 5450
+P 7150 5550
+F 0 "R5" H 7082 5504 50  0000 R CNN
+F 1 "10k" H 7082 5595 50  0000 R CNN
+F 2 "_PIC18F24K40:R_0603_1608Metric_Pad1.05x0.95mm_HandSolder" H 7150 5550 50  0001 C CNN
+F 3 "~" H 7150 5550 50  0001 C CNN
+	1    7150 5550
 	-1   0    0    1
 $EndComp
 Wire Wire Line
-	7250 5550 7250 5650
+	6700 5650 6700 5750
 $Comp
 L _PIC18F24K40:C_Small C6
 U 1 1 5BD82600
-P 8000 5850
-F 0 "C6" H 8092 5896 50  0000 L CNN
-F 1 "0.01uf" H 8092 5805 50  0000 L CNN
-F 2 "_PIC18F24K40:C_0603_1608Metric_Pad1.05x0.95mm_HandSolder" H 8000 5850 50  0001 C CNN
-F 3 "~" H 8000 5850 50  0001 C CNN
-	1    8000 5850
+P 7150 5950
+F 0 "C6" H 7242 5996 50  0000 L CNN
+F 1 "0.01uf" H 7242 5905 50  0000 L CNN
+F 2 "_PIC18F24K40:C_0603_1608Metric_Pad1.05x0.95mm_HandSolder" H 7150 5950 50  0001 C CNN
+F 3 "~" H 7150 5950 50  0001 C CNN
+	1    7150 5950
 	1    0    0    -1
 $EndComp
@@
 L _PIC18F24K40:GND #PWR05
 U 1 1 5BD82668
-P 8000 6000
-F 0 "#PWR05" H 8000 5750 50  0001 C CNN
-F 1 "GND" H 8005 5827 50  0000 C CNN
-F 2 "" H 8000 6000 50  0001 C CNN
-F 3 "" H 8000 6000 50  0001 C CNN
-	1    8000 6000
+P 7150 6100
+F 0 "#PWR05" H 7150 5850 50  0001 C CNN
+F 1 "GND" H 7155 5927 50  0000 C CNN
+F 2 "" H 7150 6100 50  0001 C CNN
+F 3 "" H 7150 6100 50  0001 C CNN
+	1    7150 6100
 	1    0    0    -1
 $EndComp
 Wire Wire Line
-	8000 6000 8000 5950
+	7150 6100 7150 6050
+Wire Wire Line
+	6700 5650 7150 5650
+Wire Wire Line
+	7150 5650 7150 5850
+Connection ~ 7150 5650
 Wire Wire Line
 	7600 5300 8000 5300
+$Comp
+L _PIC18F24K40:+5v_USB #PWR?
+U 1 1 5BDAE3BB
+P 7150 5400
+F 0 "#PWR?" H 7150 5250 50  0001 C CNN
+F 1 "+5v_USB" H 7167 5573 50  0000 C CNN
+F 2 "" H 7150 5400 50  0001 C CNN
+F 3 "" H 7150 5400 50  0001 C CNN
+	1    7150 5400
+	1    0    0    -1
+$EndComp
 Wire Wire Line
-	7250 5550 8000 5550
+	7150 5400 7150 5450
 Wire Wire Line
-	8000 5550 8000 5750
-Connection ~ 8000 5550
+	7150 5650 8000 5650
 Wire Wire Line
-	8000 5350 8000 5300
-Connection ~ 8000 5300
-Wire Wire Line
-	8000 5300 8050 5300
+	8000 5650 8000 5300
 Wire Bus Line
 	6400 5750 6400 6550
@@
 Wire Bus Line
 	3400 4100 3400 5650
+Connection ~ 8000 5300
+Wire Wire Line
+	8000 5300 8050 5300
 $EndSCHEMATC
